File: schematics/IV-27 clock.kicad_sch (KiCad schematic)
At the start: 15 parts, among them J1 BME280 module, J2 LIGHT, J3 3.3V buck, J4 25V boost, Q1 BC547, SW1 RotaryEncoder_Switch, U1 SEEEDUINO-XIAO-ESP32C3, U2 MAX6921AWI

Commit message: update schematics
Parts:
- added C1, C2: 100n, symbol Device:C
- R2, R3: value 100 -> 10
Connections:
- net G1: now also Tube-conn-right.5 (Pin_5); no longer Tube-conn-right.4 (Pin_4)
- net G10: now also Tube-conn-right.10 (Pin_10); no longer Tube-conn-right.9 (Pin_9)
- net G11: now also Tube-conn-right.7 (Pin_7); no longer Tube-conn-right.6 (Pin_6)
- net G12: now also Tube-conn-right.11 (Pin_11); no longer Tube-conn-right.10 (Pin_10)
- net G13: now also Tube-conn-right.6 (Pin_6); no longer Tube-conn-right.5 (Pin_5)
- net G14: now also Tube-conn-right.12 (Pin_12); no longer Tube-conn-right.11 (Pin_11)
- net G2: now also Tube-conn-right.4 (Pin_4); no longer Tube-conn-right.3 (Pin_3)
- net G3: now also Tube-conn-right.13 (Pin_13); no longer Tube-conn-right.12 (Pin_12)
- net G4: now also Tube-conn-right.3 (Pin_3); no longer Tube-conn-right.2 (Pin_2)
- net G8: now also Tube-conn-right.9 (Pin_9); no longer Tube-conn-right.8 (Pin_8)
- net G9: now also Tube-conn-right.8 (Pin_8); no longer Tube-conn-right.7 (Pin_7)
- net GND: now also Tube-conn-right.1 (Pin_1), C1.2, C2.2; no longer Tube-conn-right.14 (Pin_14)
- net at J3.4 (Pin_4): now also Tube-conn-right.2 (Pin_2); no longer Tube-conn-right.1 (Pin_1)
- net at SW1.A, U1.3 (PA10_A2_D2): now also C1.1
- net at SW1.B, U1.4 (PA11_A3_D3): now also C2.1
Other:
- moved on the sheet: Tube-conn-right
